File: pcb/pcb.kicad_sch (KiCad schematic)
At the start: 1 part, among them U1 ESP32-S3-WROOM-1

Commit message: a
Parts:
- added D1, D10, D11, D12, D13, D14, D15, D16, D17, D18, D19, D2, D20, D21, D22, D23, D24, D25, D26, D27, D28, D29, D3, D30, D31, D32, D33, D34, D35, D36, D37, D38, D39, D4, D40, D5, D6, D7, D8, D9: 1N4148WT, Diode_SMD:D_SOD-523, symbol Diode:1N4148WT
- added J2: USB_C_Receptacle_USB2.0_16P, Connector_USB:USB_C_Receptacle_Amphenol_124019772112A, symbol Connector:USB_C_Receptacle_USB2.0_16P
- added SW1: A, Button_Switch_Keyboard:SW_Cherry_MX_1.00u_PCB, symbol Switch:SW_Push
- added SW10: R, Button_Switch_Keyboard:SW_Cherry_MX_1.00u_PCB, symbol Switch:SW_Push
- added SW11: F, Button_Switch_Keyboard:SW_Cherry_MX_1.00u_PCB, symbol Switch:SW_Push
- added SW12: V, Button_Switch_Keyboard:SW_Cherry_MX_1.00u_PCB, symbol Switch:SW_Push
- added SW13: T, Button_Switch_Keyboard:SW_Cherry_MX_1.00u_PCB, symbol Switch:SW_Push
- added SW14: G, Button_Switch_Keyboard:SW_Cherry_MX_1.00u_PCB, symbol Switch:SW_Push
- added SW15: B, Button_Switch_Keyboard:SW_Cherry_MX_1.00u_PCB, symbol Switch:SW_Push
- added SW16: Y, Button_Switch_Keyboard:SW_Cherry_MX_1.00u_PCB, symbol Switch:SW_Push
- added SW17: H, Button_Switch_Keyboard:SW_Cherry_MX_1.00u_PCB, symbol Switch:SW_Push
- added SW18: N, Button_Switch_Keyboard:SW_Cherry_MX_1.00u_PCB, symbol Switch:SW_Push
- added SW19: 1, Button_Switch_Keyboard:SW_Cherry_MX_1.00u_PCB, symbol Switch:SW_Push
- added SW2: Q, Button_Switch_Keyboard:SW_Cherry_MX_1.00u_PCB, symbol Switch:SW_Push
- added SW20: 2, Button_Switch_Keyboard:SW_Cherry_MX_1.00u_PCB, symbol Switch:SW_Push
- added SW21: 3, Button_Switch_Keyboard:SW_Cherry_MX_1.00u_PCB, symbol Switch:SW_Push
- added SW22: 4, Button_Switch_Keyboard:SW_Cherry_MX_1.00u_PCB, symbol Switch:SW_Push
- added SW23: 5, Button_Switch_Keyboard:SW_Cherry_MX_1.00u_PCB, symbol Switch:SW_Push
- added SW24: 6, Button_Switch_Keyboard:SW_Cherry_MX_1.00u_PCB, symbol Switch:SW_Push
- added SW25: 7, Button_Switch_Keyboard:SW_Cherry_MX_1.00u_PCB, symbol Switch:SW_Push
- added SW26: U, Button_Switch_Keyboard:SW_Cherry_MX_1.00u_PCB, symbol Switch:SW_Push
- added SW27: J, Button_Switch_Keyboard:SW_Cherry_MX_1.00u_PCB, symbol Switch:SW_Push
- added SW28: ,, Button_Switch_Keyboard:SW_Cherry_MX_1.00u_PCB, symbol Switch:SW_Push
- added SW29: 8, Button_Switch_Keyboard:SW_Cherry_MX_1.00u_PCB, symbol Switch:SW_Push
- added SW3: W, Button_Switch_Keyboard:SW_Cherry_MX_1.00u_PCB, symbol Switch:SW_Push
- added SW30: I, Button_Switch_Keyboard:SW_Cherry_MX_1.00u_PCB, symbol Switch:SW_Push
- added SW31: K, Button_Switch_Keyboard:SW_Cherry_MX_1.00u_PCB, symbol Switch:SW_Push
- added SW32: ;, Button_Switch_Keyboard:SW_Cherry_MX_1.00u_PCB, symbol Switch:SW_Push
- added SW33: 9, Button_Switch_Keyboard:SW_Cherry_MX_1.00u_PCB, symbol Switch:SW_Push
- added SW34: O, Button_Switch_Keyboard:SW_Cherry_MX_1.00u_PCB, symbol Switch:SW_Push
- added SW35: L, Button_Switch_Keyboard:SW_Cherry_MX_1.00u_PCB, symbol Switch:SW_Push
- added SW36: :, Button_Switch_Keyboard:SW_Cherry_MX_1.00u_PCB, symbol Switch:SW_Push
- added SW37: 0, Button_Switch_Keyboard:SW_Cherry_MX_1.00u_PCB, symbol Switch:SW_Push
- added SW38: P, Button_Switch_Keyboard:SW_Cherry_MX_1.00u_PCB, symbol Switch:SW_Push
- added SW39: M, Button_Switch_Keyboard:SW_Cherry_MX_1.00u_PCB, symbol Switch:SW_Push
- added SW4: Z, Button_Switch_Keyboard:SW_Cherry_MX_1.00u_PCB, symbol Switch:SW_Push
- added SW40: !, Button_Switch_Keyboard:SW_Cherry_MX_1.00u_PCB, symbol Switch:SW_Push
- added SW5: S, Button_Switch_Keyboard:SW_Cherry_MX_1.00u_PCB, symbol Switch:SW_Push
- added SW6: X, Button_Switch_Keyboard:SW_Cherry_MX_1.00u_PCB, symbol Switch:SW_Push
- added SW7: E, Button_Switch_Keyboard:SW_Cherry_MX_1.00u_PCB, symbol Switch:SW_Push
- added SW8: D, Button_Switch_Keyboard:SW_Cherry_MX_1.00u_PCB, symbol Switch:SW_Push
- added SW9: C, Button_Switch_Keyboard:SW_Cherry_MX_1.00u_PCB, symbol Switch:SW_Push
- added U14: MAX604, symbol Regulator_Linear:MAX604
Connections:
- net GND: now reaches U1.1 (GND), U1.40 (GND), U1.41 (GND)
- net GND: now also J2.A1 (GND), J2.A12 (GND), J2.B1 (GND), J2.B12 (GND)
- net D-: now reaches U1.13 (USB_D-)
- net D-: now also J2.A7 (D-), J2.B7 (D-)
- net D+: now reaches U1.14 (USB_D+)
- net D+: now also J2.A6 (D+), J2.B6 (D+)
- net +3.3V: now reaches U1.2 (3V3)
- new net: D7.2 (A), SW7.2
- new net: D17.2 (A), SW17.2
- new net: D25.2 (A), SW25.2
- new net: D10.2 (A), SW10.2
- new net: D31.2 (A), SW31.2
- new net: D38.2 (A), SW38.2
- new net: D39.2 (A), SW39.2
- new net: D32.2 (A), SW32.2
- new net: D36.2 (A), SW36.2
- new net: D27.2 (A), SW27.2
- new net: D6.2 (A), SW6.2
- new net: D30.2 (A), SW30.2
- new net: D2.2 (A), SW2.2
- new net: D3.2 (A), SW3.2
- new net: D16.2 (A), SW16.2
- new net: D5.2 (A), SW5.2
- new net: D37.2 (A), SW37.2
- new net: D12.2 (A), SW12.2
- new net: D40.2 (A), SW40.2
- new net: D26.2 (A), SW26.2
- new net: D22.2 (A), SW22.2
- new net: D20.2 (A), SW20.2
- new net: D34.2 (A), SW34.2
- new net: D23.2 (A), SW23.2
- new net: D1.2 (A), SW1.2
- new net: D11.2 (A), SW11.2
- new net: D35.2 (A), SW35.2
- new net: D4.2 (A), SW4.2
- new net: D28.2 (A), SW28.2
- new net: D33.2 (A), SW33.2
- new net: D18.2 (A), SW18.2
- new net: D8.2 (A), SW8.2
- new net: D21.2 (A), SW21.2
- new net: D15.2 (A), SW15.2
- new net: D24.2 (A), SW24.2
- new net: U14.2 (GND), U14.3 (GND), U14.6 (GND), U14.7 (GND)
- new net: D19.2 (A), SW19.2
- new net: D9.2 (A), SW9.2
- new net: D13.2 (A), SW13.2
- new net: D14.2 (A), SW14.2
- new net: D29.2 (A), SW29.2
- new net Col1: D1.1 (K), D19.1 (K), D2.1 (K), D3.1 (K)
- new net Col10: D37.1 (K), D38.1 (K), D39.1 (K), D40.1 (K)
- new net Col2: D20.1 (K), D4.1 (K), D5.1 (K), D6.1 (K)
- new net Col3: D21.1 (K), D7.1 (K), D8.1 (K), D9.1 (K)
- new net Col4: D10.1 (K), D11.1 (K), D12.1 (K), D22.1 (K)
- new net Col5: D13.1 (K), D14.1 (K), D15.1 (K), D23.1 (K)
- new net Col6: D16.1 (K), D17.1 (K), D18.1 (K), D24.1 (K)
- new net Col7: D25.1 (K), D26.1 (K), D27.1 (K), D28.1 (K)
- new net Col8: D29.1 (K), D30.1 (K), D31.1 (K), D32.1 (K)
- new net Col9: D33.1 (K), D34.1 (K), D35.1 (K), D36.1 (K)
- new net L1: SW19.1, SW20.1, SW21.1, SW22.1, SW23.1, SW24.1, SW25.1, SW29.1, SW33.1, SW37.1
- new net L2: SW1.1, SW10.1, SW13.1, SW16.1, SW26.1, SW30.1, SW34.1, SW38.1, SW4.1, SW7.1
- new net L3: SW11.1, SW14.1, SW17.1, SW2.1, SW27.1, SW31.1, SW35.1, SW39.1, SW5.1, SW8.1
- new net L4: SW12.1, SW15.1, SW18.1, SW28.1, SW3.1, SW32.1, SW36.1, SW40.1, SW6.1, SW9.1
- new net Vusb: J2.A4 (VBUS), J2.A9 (VBUS), J2.B4 (VBUS), J2.B9 (VBUS)
- no-connect marks 0 -> 5
