File: Recepteur/Dongle/PCB.kicad_pcb (KiCad board)
At the start: 2 copper layers, 21 x 45 mm, 14 parts, among them J1 USB_A, J2 Conn_01x07, SW3 SW_Push, SW4 SW_Push, U2 MAX604, X1 ESP32-S3-WROOM-1-N16R8

Commit message: update schema & pcb
Parts:
- removed J2: Conn_01x07, Connector_PinHeader_2.54mm:PinHeader_1x07_P2.54mm_Vertical
- removed U2: MAX604, Package_SO:SOIC-8-N7_3.9x4.9mm_P1.27mm
- removed X1: ESP32-S3-WROOM-1-N16R8, ESP32-S3-WROOM-1-N16R8:ESP32S3WROOM1N8R2
- added U3: ESP32-S3-MINI-1, RF_Module:ESP32-S2-MINI-1, B.Cu at (177.4, 94.7)
- added U4: TLV75533PDBV, Package_TO_SOT_SMD:SOT-23-5, F.Cu at (182.1, 101.0)
- C1, C2: value 10µ -> 1µ
- SW3, SW4: footprint Button_Switch_SMD:Panasonic_EVQPUL_EVQPUC -> Button_Switch_SMD:SW_Tactile_SPST_NO_Straight_CK_PTS636Sx25SMTRLFS
- moved SW4 77.9 mm to (172.0, 98.0), turned to -90 degrees
- moved R5 77.2 mm to (174.5, 102.5), turned to 180 degrees
- moved C1 73.0 mm to (179.1, 101.9), turned to -90 degrees
- moved D5 71.3 mm to (177.2, 101.7), turned to 90 degrees
- moved C2 69.9 mm to (182.3, 105.2), turned to 0 degrees
- moved J1 69.8 mm to (177.4, 117.5)
- moved R2 67.3 mm to (176.4, 98.3), turned to -90 degrees
- moved SW3 65.4 mm to (177.7, 93.7), turned to 0 degrees
- moved R4 65.0 mm to (178.5, 98.3), turned to 90 degrees
- moved R3 60.6 mm to (182.3, 97.2), turned to 90 degrees
- moved D4 59.6 mm to (184.2, 97.2), turned to 90 degrees
Connections:
- net V+ renamed 5V
Routing:
- net 5V: track 24.7 -> 9.07 mm, vias 2 -> 0
- net D+: track 15.3 -> 3.90 mm
- net D-: track 16.2 -> 4.94 mm
- net +3.3V: track 29.8 -> 19.5 mm
- net GND: track 14.4 -> 5.22 mm
- net EN (Reset): track 19.3 -> 13.5 mm
- net BOOT: track 15.0 -> 9.88 mm
- net Net-(D4-A): track 3.51 -> 1.96 mm
- net Net-(D5-A): track 3.21 -> 2.00 mm
Other:
- board size 21 x 45 mm -> 17.5 x 24.8 mm
