File: Electronique/Clavier/pcb.kicad_pcb (KiCad board)
At the start: 2 copper layers, 130 parts, among them SW1 A, SW10 R, SW11 F, SW12 C, SW13 T, SW14 G, SW15 V, SW16 Y, SW17 H, SW18 B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

Commit message: edit schema
Parts:
- moved SW47 41.0 mm to (263.5, -14.9)
- moved SW43 40.1 mm to (263.5, 4.13)
- moved SW48 32.5 mm to (282.7, -14.9)
- moved SW46 16.5 mm to (358.0, 146.9)
