File: Electronique/Clavier/pcb.kicad_pcb (KiCad board)
At the start: 2 copper layers, 170 parts, among them J3 Conn_01x05, Q3 BSS84, Q4 BSS138, SW1 A, SW10 R, SW11 F, SW12 C, SW13 T, SW14 G, SW15 V, SW16 Y, SW17 H, SW18 B, SW19 1, SW2 Q, SW20 2, SW21 3, SW22 4, SW23 5, SW24 6, SW25 7, SW26 U, SW27 J, SW28 N, SW29 8, SW3 <, SW30 I, SW31 K, SW32 ,, SW33 9, SW34 O, SW35 L, SW36 ;, SW37 0, SW38 P, SW39 M, SW4 Z, SW40 :, SW41 SW_Push, SW42 SW_Push, SW43 ², SW44 Tab, SW45 VMaj, SW46 Shift, SW47 Echap, SW48 F1, SW49 F2, SW5 S, SW50 F3, SW51 F4, SW52 F5, SW53 F6, SW54 F7, SW55 F8, SW56 F9, SW57 F10, SW58 F11, SW59 ), SW6 W, SW60 ^, SW61 ù, SW62 !, SW63 F12, SW64 =, SW65 $, SW66 *, SW67 Up, SW7 E, SW8 D, SW9 X, U1 ESP32-S3-WROOM-1, U3 USBLC6-2P6, U4 TLV75533PDBV, U6 MCP73871-2CC

Commit message: m
Parts:
- removed D49, D50, D51, D52, D53, D54, D55, D56, D57, D58: 1N4148WT, Diode_SMD:D_SOD-523
- removed J3: Conn_01x05, Connector_PinHeader_2.54mm:PinHeader_1x05_P2.54mm_Vertical
- removed SW52: F5, Library:SW_Cherry_MX_1.00u_PCB
- removed SW53: F6, Library:SW_Cherry_MX_1.00u_PCB
- removed SW54: F7, Library:SW_Cherry_MX_1.00u_PCB
- removed SW55: F8, Library:SW_Cherry_MX_1.00u_PCB
- removed SW56: F9, Library:SW_Cherry_MX_1.00u_PCB
- removed SW57: F10, Library:SW_Cherry_MX_1.00u_PCB
- removed SW58: F11, Library:SW_Cherry_MX_1.00u_PCB
- removed SW63: F12, Library:SW_Cherry_MX_1.00u_PCB
- added C10: 10n, Capacitor_SMD:C_0603_1608Metric_Pad1.08x0.95mm_HandSolder, B.Cu at (-202.9, -69.0)
- added C14: 10n, Capacitor_SMD:C_0603_1608Metric_Pad1.08x0.95mm_HandSolder, B.Cu at (-208.3, -57.2)
- added C15: 10n, Capacitor_SMD:C_0603_1608Metric_Pad1.08x0.95mm_HandSolder, B.Cu at (-197.5, -57.2)
- added C9: 4,7nF, Capacitor_SMD:C_0603_1608Metric_Pad1.08x0.95mm_HandSolder, F.Cu at (-188.1, -60.0)
- added D41: 1N4148WT, Diode_SMD:D_SOD-523, F.Cu at (113.7, -27.4)
- added D63: 1N4148WT, Diode_SMD:D_SOD-523, F.Cu at (89.0, -95.7)
- added D68: 1N4148WT, Diode_SMD:D_SOD-523, F.Cu at (113.7, -62.0)
- added D70: 1N4148WT, Diode_SMD:D_SOD-523, B.Cu at (92.7, -32.2)
- added D74: 1N4148WT, Diode_SMD:D_SOD-523, B.Cu at (-170.1, -2.29)
- added D75: 1N4148WT, Diode_SMD:D_SOD-523, B.Cu at (-139.8, -6.82)
- added D76: 1N4148WT, Diode_SMD:D_SOD-523, B.Cu at (-122.5, -5.51)
- added D77: 1N4148WT, Diode_SMD:D_SOD-523, B.Cu at (-54.1, -8.26)
- added D83: 1N4148WT, Diode_SMD:D_SOD-523, B.Cu at (38.2, -10.5)
- added D85: 1N4148WT, Diode_SMD:D_SOD-523, B.Cu at (76.3, -11.8)
- added D86: 1N4148WT, Diode_SMD:D_SOD-523, B.Cu at (93.7, -13.0)
- added D87: 1N4148WT, Diode_SMD:D_SOD-523, F.Cu at (113.7, -8.87)
- added Q5: FS8205A, Package_SO:SOP65P640X120-8N, F.Cu at (-188.7, -69.7)
- added R1: 10K, Resistor_SMD:R_0805_2012Metric, F.Cu at (-195.4, -89.3)
- added R12: 100, Resistor_SMD:R_0805_2012Metric, F.Cu at (-191.9, -62.1)
- added R13: 1k, Resistor_SMD:R_0805_2012Metric, F.Cu at (-189.1, -66.8)
- added R14: 200, Resistor_SMD:R_0805_2012Metric, B.Cu at (-207.0, -68.9)
- added R15: 200, Resistor_SMD:R_0805_2012Metric, B.Cu at (-204.9, -68.9)
- added R24: 200, Resistor_SMD:R_0805_2012Metric, B.Cu at (-198.9, -68.9)
- added R25: 10k, Resistor_SMD:R_0805_2012Metric, B.Cu at (-201.1, -68.9)
- added R26: 10k, Resistor_SMD:R_0805_2012Metric, B.Cu at (-205.4, -60.7)
- added R27: 10k, Resistor_SMD:R_0805_2012Metric, B.Cu at (-200.4, -60.7)
- added SW68: SW_Push_SPDT, Button_Switch_THT:SW_Slide-03_Wuerth-WS-SLTV_10x2.5x6.4_P2.54mm, F.Cu at (-189.9, -56.5)
- added SW70: Delete, Library:SW_Cherry_MX_Plate_1.00u, F.Cu at (83.8, -76.0)
- added SW71: Entrer, Library:SW_Cherry_MX_Plate_1.75u, F.Cu at (100.4, -56.9)
- added SW73: Up, Library:SW_Cherry_MX_Plate_1.00u, F.Cu at (88.5, -18.8)
- added SW74: CTRL, Library:SW_Cherry_MX_Plate_1.25u, F.Cu at (-161.5, 0.23)
- added SW75: Win, Library:SW_Cherry_MX_Plate_1.25u, F.Cu at (-137.7, 0.23)
- added SW76: Alt, Library:SW_Cherry_MX_Plate_1.25u, F.Cu at (-113.9, 0.23)
- added SW77: Space, Library:SW_Cherry_MX_Plate_6.25u, F.Cu at (-42.5, 0.23)
- added SW83: Fn, Library:SW_Cherry_MX_Plate_1.25u, F.Cu at (29.0, 0.23)
- added SW85: Left, Library:SW_Cherry_MX_Plate_1.00u, F.Cu at (69.5, 0.23)
- added SW86: Down, Library:SW_Cherry_MX_Plate_1.00u, F.Cu at (88.5, 0.23)
- added SW87: Right, Library:SW_Cherry_MX_Plate_1.00u, F.Cu at (107.6, 0.23)
- added U2: DW01A, Package_TO_SOT_SMD:SOT-23-6, F.Cu at (-188.2, -63.2)
- added U5: ~, Battery:Lipo1s, F.Cu at (-191.9, -19.4)
- C11, C12, C2, C3, C5, D1, D10, D11, D12, D13, D14, D15, D16, D17, D18, D19, D2, D20, D21, D22, D23, D24, D25, D26, D27, D28, D3, D30, D31, D32, D34, D35, D36, D38, D39, D4, D40, D42, D43, D44, D45, D46, D5, D6, D60, D61, D62, D65, D66, D67, D7, D72, D73, D8, D9, R16, R17, R18, R20, R21, R22, R23, R4, R5, SW41, SW42, U4, U6: moved to B.Cu
- C4: value 100nF -> 100n; moved to F.Cu
- Q3, Q4, R7, R8, R9, U1: moved to F.Cu
- SW1, SW10, SW11, SW12, SW13, SW14, SW15, SW16, SW17, SW18, SW19, SW2, SW20, SW21, SW22, SW23, SW24, SW25, SW26, SW27, SW28, SW29, SW3, SW30, SW31, SW32, SW33, SW34, SW35, SW36, SW37, SW38, SW39, SW4, SW40, SW43, SW5, SW59, SW6, SW60, SW61, SW62, SW64, SW65, SW66, SW7, SW8, SW9: footprint Library:SW_Cherry_MX_1.00u_PCB -> Library:SW_Cherry_MX_Plate_1.00u
- SW44: footprint Library:SW_Cherry_MX_1.00u_PCB -> Library:SW_Cherry_MX_Plate_1.50u
- SW45: footprint Library:SW_Cherry_MX_1.00u_PCB -> Library:SW_Cherry_MX_Plate_2.00u
- SW46: footprint Library:SW_Cherry_MX_1.00u_PCB -> Library:SW_Cherry_MX_Plate_1.25u
- SW47: value Echap -> PageDown; footprint Library:SW_Cherry_MX_1.00u_PCB -> Library:SW_Cherry_MX_Plate_1.00u
- SW48: value F1 -> DEF; footprint Library:SW_Cherry_MX_1.00u_PCB -> Library:SW_Cherry_MX_Plate_1.00u
- SW49: value F2 -> Definir; footprint Library:SW_Cherry_MX_1.00u_PCB -> Library:SW_Cherry_MX_Plate_1.25u
- SW50: value F3 -> Definir; footprint Library:SW_Cherry_MX_1.00u_PCB -> Library:SW_Cherry_MX_Plate_1.25u
- SW51: value F4 -> COM-15141; footprint Library:SW_Cherry_MX_1.00u_PCB -> Rotary_Encoder:COM-15141_SPK
- SW67: value Up -> PageUp; footprint Library:SW_Cherry_MX_1.00u_PCB -> Library:SW_Cherry_MX_Plate_1.00u
- moved C6 561.7 mm to (-199.1, -98.2)
- moved C8 560.9 mm to (-196.4, -98.1)
- moved SW42 560.9 mm to (-182.4, -95.1), turned to -90 degrees
- moved C7 556.9 mm to (-189.2, -94.5), turned to -90 degrees
- moved C3 556.8 mm to (-190.2, -98.1)
- moved C2 556.4 mm to (-188.0, -98.1)
- moved U4 555.8 mm to (-196.5, -98.2)
- moved C5 551.9 mm to (-195.9, -94.7), turned to -45 degrees
- moved R5 551.3 mm to (-178.4, -91.2), turned to 180 degrees
- moved Q4 549.0 mm to (-197.5, -80.5)
- moved C12 548.0 mm to (-204.0, -85.2), turned to 180 degrees
- moved U1 547.1 mm to (-184.5, -93.3), turned to 0 degrees
- moved R22 546.3 mm to (-203.6, -89.6), turned to 0 degrees
- moved R9 546.2 mm to (-200.3, -76.3), turned to 90 degrees
- moved C11 545.9 mm to (-203.6, -79.8)
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Connections:
- D42 pad 1: Col13 -> Col12
- D47 pad 1: Col1 -> Col15
- D48 pad 1: Col2 -> Col15
- D71 pad 1: Net-(D71-K) -> PG
- J1 pad 1: GND -> Vbat-
- J1 pad 2: Vbat -> Vbat_Mes
- J2 pad S1: unconnected-(J2-SHIELD-PadS1)_2 -> GND
- Q3 pad 2: Vbat -> Vbat_Mes
- R9 pad 1: Vbat -> Vbat_Mes
- SW47 pad 1: L1 -> L4
- SW47 pad 2: Net-(D47-A) -> Net-(D41-A)
- SW48 pad 1: L1 -> L5
- SW48 pad 2: Net-(D48-A) -> Net-(D42-A)
- SW49 pad 2: Net-(D49-A) -> Net-(D48-A)
- SW50 pad 1: L1 -> L3
- SW50 pad 2: Net-(D50-A) -> Net-(D47-A)
- SW51 pad 1: L1 -> Net-(R14-Pad2)
- U1 pad 13: D- -> DP-
- U1 pad 14: D+ -> DP+
- U1 pad 15: unconnected-(U1-IO3-Pad15) -> Check Batt En
- U1 pad 16: unconnected-(U1-IO46-Pad16) -> Check Batt
- U1 pad 17: unconnected-(U1-IO9-Pad17) -> L5
- U1 pad 31: unconnected-(U1-IO38-Pad31) -> Col9
- U1 pad 32: unconnected-(U1-IO39-Pad32) -> Col10
- U1 pad 33: unconnected-(U1-IO40-Pad33) -> Col11
- U1 pad 34: unconnected-(U1-IO41-Pad34) -> Col12
- U1 pad 35: unconnected-(U1-IO42-Pad35) -> Col13
- U1 pad 38: Check Batt En -> Col14
- U1 pad 39: Check Batt -> Col15
- U1 pad 9: unconnected-(U1-IO16-Pad9) -> PG
- U3 pad 1: D+ -> D-
- U3 pad 3: unconnected-(U3-I/O2-Pad3) -> D+
- U3 pad 4: unconnected-(U3-I/O2-Pad4) -> DP+
- U3 pad 6: D- -> DP-
- U6 pad 6: Net-(D71-K) -> PG
Routing:
- net Col15: track 0.00 -> 376.9 mm
- net Col14: track 0.00 -> 351.9 mm, vias 0 -> 1
- net Col13: track 0.00 -> 340.5 mm, vias 0 -> 1
- net Col12: track 0.00 -> 322.3 mm, vias 0 -> 1
- net Col11: track 0.00 -> 303.9 mm, vias 0 -> 1
- net L5: track 0.00 -> 269.1 mm
- net Col10: track 0.00 -> 259.0 mm, vias 0 -> 1
- net Col9: track 0.00 -> 235.2 mm, vias 0 -> 1
- net L1: track 460.8 -> 269.1 mm
- net Col2: track 0.00 -> 71.9 mm
- net Col3: track 0.00 -> 67.9 mm
- net Col1: track 0.00 -> 65.3 mm
- net Col6: track 0.00 -> 62.0 mm
- net Col4: track 0.00 -> 49.6 mm
- net L2: track 211.8 -> 259.6 mm
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Other:
- board outline added: 351.1 x 120.4 mm
- copper layers 2 -> 4
