File: Electronique/Clavier/pcb.kicad_sch (KiCad schematic)
At the start: 137 parts, among them SW1 A, SW10 R, SW11 F, SW12 C, SW13 T, SW14 G, SW15 V, SW16 Y, SW17 H, SW18 B, SW19 1, SW2 Q, SW20 2, SW21 3, SW22 4, SW23 5, SW24 6, SW25 7, SW26 U, SW27 J, SW28 N, SW29 8, SW3 <, SW30 I, SW31 K, SW32 ,, SW33 9, SW34 O, SW35 L, SW36 ;, SW37 0, SW38 P, SW39 M, SW4 Z, SW40 :, SW41 SW_Push, SW42 SW_Push, SW43 ², SW44 Tab, SW45 VMaj, SW46 Shift, SW47 Echap, SW48 F1, SW49 F2, SW5 S, SW50 F3, SW51 F4, SW52 F5, SW53 F6, SW54 F7, SW55 F8, SW56 F9, SW57 F10, SW58 F11, SW59 ), SW6 W, SW60 ^, SW61 ù, SW62 !, SW7 E, SW8 D, SW9 X, U1 ESP32-S3-WROOM-1, U14 MAX604, U2 MCP73831-2-MC

Commit message: edit schema
Parts:
- removed C3, C4: 10µF, symbol Device:C
- removed U14: MAX604, symbol Regulator_Linear:MAX604
- added C5, C6: 10µ, Capacitor_SMD:C_0603_1608Metric_Pad1.08x0.95mm_HandSolder, symbol Device:C
- added Q1, Q3: BSS84, Package_TO_SOT_SMD:SOT-23, symbol Transistor_FET:BSS84
- added Q4: BSS138, Package_TO_SOT_SMD:SOT-23, symbol Transistor_FET:BSS138
- added R10, R8, R9: 100k, Resistor_SMD:R_0805_2012Metric, symbol Device:R
- added R3, R6: 5.1k, Resistor_SMD:R_0805_2012Metric, symbol Device:R
- added R7: 220k, Resistor_SMD:R_0805_2012Metric, symbol Device:R
- added SW63: RotaryEncoder_Switch, symbol Device:RotaryEncoder_Switch
- added U4: TLV75533PDBV, Package_TO_SOT_SMD:SOT-23-5, symbol Regulator_Linear:TLV75533PDBV
- R1, R2: footprint (none) -> Resistor_SMD:R_0805_2012Metric
Connections:
- net +3.3V: now also C6.1, U4.5 (OUT)
- net GND: now also C5.2, C6.2, Q4.2 (S), R10.2, R3.2, R6.2, R7.2, U4.2 (GND)
- net Vbat: now also Q1.3 (D), Q3.2 (S), R9.1; no longer D42.1 (K)
- net Vusb: now also Q1.1 (G), R10.1
- net at J2.A5 (CC1): now also R3.1
- net at J2.B5 (CC2): now also R6.1
- net Check Batt En: now reaches U1.38 (IO2)
- net Check Batt En: now also Q4.1 (G)
- net Check Batt: now reaches U1.39 (IO1)
- net Check Batt: now also R7.1, R8.2
- new net: C5.1, D42.1 (K), Q1.2 (S), U4.1 (IN), U4.3 (EN)
- new net: Q3.1 (G), Q4.3 (D), R9.2
- new net: Q3.3 (D), R8.1
- no-connect marks 5 -> 3
Other:
- note added: "Circuit de vérification de la capacité de la batterie L'ADC de l'ESP32 étant limité à une tension de 3,3V, un PDT par 0,68 est utilisé pour ramener la tension batterie (max 4,2V) à 2,88v max. Le transistor NMOS est controlé par le µC pour décider quand on veut vérifier la capacité de la batterie. Le transistor PMOS coupe l'alimentation du PDT et est controlé par le NMOS, donc le µC, évitant ainsi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"
- note added: "Encodeur - Volume"
- note added: "Indicateur de batterie"
- note added: "Note : Le régulateur TLV75533PDBV à un dropout Maximum de 238mV, il faut donc qu'il soit alimenté au minimum en 3v5 pour fournir du 3v3."
- note added: "Régulateur 3v3 + Commutateur d'alimentation"
- note removed: "Regulateur de tension"
- moved on the sheet: C1, C2, D41, D42, J1, R1, R2
