File: Electronique/Clavier/pcb.kicad_sch (KiCad schematic)
At the start: 174 parts, among them J3 Conn_01x05, Q3 BSS84, Q4 BSS138, SW1 A, SW10 R, SW11 F, SW12 C, SW13 T, SW14 G, SW15 V, SW16 Y, SW17 H, SW18 B, SW19 1, SW2 Q, SW20 2, SW21 3, SW22 4, SW23 5, SW24 6, SW25 7, SW26 U, SW27 J, SW28 N, SW29 8, SW3 <, SW30 I, SW31 K, SW32 ,, SW33 9, SW34 O, SW35 L, SW36 ;, SW37 0, SW38 P, SW39 M, SW4 Z, SW40 :, SW41 SW_Push, SW42 SW_Push, SW43 ², SW44 Tab, SW45 VMaj, SW46 Shift, SW47 Echap, SW48 F1, SW49 F2, SW5 S, SW50 F3, SW51 F4, SW52 F5, SW53 F6, SW54 F7, SW55 F8, SW56 F9, SW57 F10, SW58 F11, SW59 ), SW6 W, SW60 ^, SW61 ù, SW62 !, SW63 F12, SW64 =, SW65 $, SW66 *, SW67 Up, SW68 SW_Push_SPDT, SW7 E, SW8 D, SW9 X, U1 ESP32-S3-WROOM-1, U3 USBLC6-2P6, U4 TLV75533PDBV, U6 MCP73871-2CC

Commit message: m
Parts:
- removed D49, D50, D51, D52, D53, D54, D55, D56, D57, D58: 1N4148WT, Diode_SMD:D_SOD-523, symbol Diode:1N4148WT
- removed J3: Conn_01x05, Connector_PinHeader_2.54mm:PinHeader_1x05_P2.54mm_Horizontal, symbol Connector_Generic:Conn_01x05
- removed SW51: F4, Library:SW_Cherry_MX_1.00u_PCB, symbol Switch:SW_Push
- removed SW52: F5, Library:SW_Cherry_MX_1.00u_PCB, symbol Switch:SW_Push
- removed SW53: F6, Library:SW_Cherry_MX_1.00u_PCB, symbol Switch:SW_Push
- removed SW54: F7, Library:SW_Cherry_MX_1.00u_PCB, symbol Switch:SW_Push
- removed SW55: F8, Library:SW_Cherry_MX_1.00u_PCB, symbol Switch:SW_Push
- removed SW56: F9, Library:SW_Cherry_MX_1.00u_PCB, symbol Switch:SW_Push
- removed SW57: F10, Library:SW_Cherry_MX_1.00u_PCB, symbol Switch:SW_Push
- removed SW58: F11, Library:SW_Cherry_MX_1.00u_PCB, symbol Switch:SW_Push
- removed SW63: F12, Library:SW_Cherry_MX_1.00u_PCB, symbol Switch:SW_Push
- added C14, C15: 10n, Capacitor_SMD:C_0603_1608Metric_Pad1.08x0.95mm_HandSolder, symbol Device:C
- added D41, D63, D68, D70, D74, D75, D76, D77, D83, D85, D86, D87: 1N4148WT, Diode_SMD:D_SOD-523, symbol Diode:1N4148WT
- added Q5: FS8205A, Package_SO:SOP65P640X120-8N, symbol FS8205A:FS8205A
- added R12: 100, Resistor_SMD:R_0805_2012Metric, symbol Device:R
- added R13: 1k, Resistor_SMD:R_0805_2012Metric, symbol Device:R
- added R14, R15, R24: 200, Resistor_SMD:R_0805_2012Metric, symbol Device:R
- added R25, R26, R27: 10k, Resistor_SMD:R_0805_2012Metric, symbol Device:R
- added SW51: COM-15141, COM-15141_SPK, symbol COM-15141:COM-15141
- added SW70: Delete, Library:SW_Cherry_MX_Plate_1.00u, symbol Switch:SW_Push
- added SW71: Entrer, Library:SW_Cherry_MX_Plate_1.75u, symbol Switch:SW_Push
- added SW73: Up, Library:SW_Cherry_MX_Plate_1.00u, symbol Switch:SW_Push
- added SW74: CTRL, Library:SW_Cherry_MX_Plate_1.25u, symbol Switch:SW_Push
- added SW75: Win, Library:SW_Cherry_MX_Plate_1.25u, symbol Switch:SW_Push
- added SW76: Alt, Library:SW_Cherry_MX_Plate_1.25u, symbol Switch:SW_Push
- added SW77: Space, Library:SW_Cherry_MX_Plate_6.25u, symbol Switch:SW_Push
- added SW83: Fn, Library:SW_Cherry_MX_Plate_1.25u, symbol Switch:SW_Push
- added SW85: Left, Library:SW_Cherry_MX_Plate_1.00u, symbol Switch:SW_Push
- added SW86: Down, Library:SW_Cherry_MX_Plate_1.00u, symbol Switch:SW_Push
- added SW87: Right, Library:SW_Cherry_MX_Plate_1.00u, symbol Switch:SW_Push
- added U2: DW01A, Package_TO_SOT_SMD:SOT-23-6, symbol Battery_Management:DW01A
- added U5: ~, Battery:Lipo1s, symbol New_Library_0:Lipo1s
- C10: value 10nF -> 10n
- C4: value 100nF -> 100n
- C9: value 10nF -> 4,7nF
- R1: footprint (none) -> Resistor_SMD:R_0805_2012Metric
- SW1, SW10, SW11, SW12, SW13, SW14, SW15, SW16, SW17, SW18, SW19, SW2, SW20, SW21, SW22, SW23, SW24, SW25, SW26, SW27, SW28, SW29, SW3, SW30, SW31, SW32, SW33, SW34, SW35, SW36, SW37, SW38, SW39, SW4, SW40, SW43, SW5, SW59, SW6, SW60, SW61, SW62, SW64, SW65, SW66, SW7, SW8, SW9: footprint Library:SW_Cherry_MX_1.00u_PCB -> Library:SW_Cherry_MX_Plate_1.00u
- SW44: footprint Library:SW_Cherry_MX_1.00u_PCB -> Library:SW_Cherry_MX_Plate_1.50u
- SW45: footprint Library:SW_Cherry_MX_1.00u_PCB -> Library:SW_Cherry_MX_Plate_2.00u
- SW46: footprint Library:SW_Cherry_MX_1.00u_PCB -> Library:SW_Cherry_MX_Plate_1.25u
- SW47: value Echap -> PageDown; footprint Library:SW_Cherry_MX_1.00u_PCB -> Library:SW_Cherry_MX_Plate_1.00u
- SW48: value F1 -> DEF; footprint Library:SW_Cherry_MX_1.00u_PCB -> Library:SW_Cherry_MX_Plate_1.00u
- SW49: value F2 -> Definir; footprint Library:SW_Cherry_MX_1.00u_PCB -> Library:SW_Cherry_MX_Plate_1.25u
- SW50: value F3 -> Definir; footprint Library:SW_Cherry_MX_1.00u_PCB -> Library:SW_Cherry_MX_Plate_1.25u
- SW67: value Up -> PageUp; footprint Library:SW_Cherry_MX_1.00u_PCB -> Library:SW_Cherry_MX_Plate_1.00u
- SW68: footprint (none) -> Button_Switch_THT:SW_Slide-03_Wuerth-WS-SLTV_10x2.5x6.4_P2.54mm
Connections:
- net DT is gone; now on net GND: C10.1
- net +3.3V: now also R26.2, R27.2, SW51.5
- net Check Batt: now also U1.16 (IO46); no longer U1.39 (IO1)
- net Check Batt En: now also U1.15 (IO3); no longer U1.38 (IO2)
- net Col1: now also U1.19 (IO11), D74.1 (K); no longer D47.1 (K)
- net Col10: now also U1.32 (IO39)
- net Col11: now also U1.33 (IO40), D83.1 (K)
- net Col12: now also D42.1 (K), U1.34 (IO41)
- net Col13: now also U1.35 (IO42), D85.1 (K); no longer D42.1 (K)
- net Col2: now also U1.20 (IO12), D75.1 (K); no longer D48.1 (K)
- net Col3: now also U1.21 (IO13), D76.1 (K)
- net Col4: now also U1.22 (IO14)
- net Col5: now also U1.8 (IO15)
- net Col6: now also U1.10 (IO17), D77.1 (K)
- net Col7: now also U1.11 (IO18)
- net Col8: now also U1.23 (IO21)
- net Col9: now also U1.31 (IO38)
- net D+: now also U3.3 (I/O2); no longer U1.14 (USB_D+), U3.1 (I/O1)
- net D-: now also U3.1 (I/O1); no longer U1.13 (USB_D-), U3.6 (I/O1)
- net GND: now also C14.1, C15.1, Q5.1, Q5.6, Q5.7, Q5.8, R13.2, R25.1, SW51.C; no longer C10.2, C9.2, J1.1 (Pin_1)
- net L1: now also U1.6 (IO6), SW70.1; no longer SW47.1, SW48.1, SW50.1
- net L2: now also U1.7 (IO7), SW71.1
- net L3: now also SW50.1, U1.12 (IO8)
- net L4: now also SW47.1, U1.18 (IO10), SW73.1
- net PG: now also U1.4 (IO4); no longer U1.9 (IO16)
- net Vbat: now also R12.1; no longer Q3.2 (S), R9.1
- net at D48.2 (A): now also SW49.2; no longer SW48.2
- net at D42.2 (A): now also SW48.2
- net at SW50.2: now also D47.2 (A)
- net Vbat_Mes: now reaches J1.2 (Pin_2), SW68.2 (B)
- net Vbat_Mes: now also Q3.2 (S), R9.1
- net at SW47.2: now also D41.2 (A); no longer D47.2 (A)
- net DP+: now reaches U3.4 (I/O2)
- net DP+: now also U1.14 (USB_D+)
- net L5: now reaches U1.17 (IO9)
- net L5: now also SW48.1, SW74.1, SW75.1, SW76.1, SW77.1, SW83.1, SW85.1, SW86.1, SW87.1
- net Vol_Down: now reaches U1.24 (IO47)
- net Vol_Down: now also C15.2, R27.1, SW51.B
- net Vol_Up: now reaches U1.25 (IO48)
- net Vol_Up: now also C14.2, R26.1, SW51.A
- net Mute_btn: now reaches U1.26 (IO45)
- net Mute_btn: now also C10.2, R25.2, SW51.3
- net CLK renamed Vbat-
- net Vbat-: now also J1.1 (Pin_1), Q5.2, Q5.3, U2.6 (GND)
- new net: C9.2, R12.2, U2.5 (VCC)
- new net: R13.1, U2.2 (CS)
- new net: R14.2, SW51.1
- new net: R15.2, SW51.2
- new net: R24.1, SW51.4
- new net: D76.2 (A), SW76.2
- new net: D85.2 (A), SW85.2
- new net: D68.2 (A), SW71.2
- new net: D74.2 (A), SW74.2
- new net: D70.2 (A), SW73.2
- new net: D75.2 (A), SW75.2
- new net: D86.2 (A), SW86.2
- new net: D63.2 (A), SW70.2
- new net: D77.2 (A), SW77.2
- new net: D83.2 (A), SW83.2
- new net: Q5.4, U2.1 (OD)
- new net: Q5.5, U2.3 (OC)
- new net: D87.2 (A), SW87.2
- new net Col14: D63.1 (K), D70.1 (K), D86.1 (K), U1.38 (IO2)
- new net Col15: D41.1 (K), D47.1 (K), D48.1 (K), D68.1 (K), D87.1 (K), U1.39 (IO1)
- new net DP-: U1.13 (USB_D-), U3.6 (I/O1)
Other:
- note added: "Protection de batterie avec un BMS"
- note added: "Régulateur 3v3"
- note removed: "Régulateur 3v3 + Commutateur d'alimentation"
- moved on the sheet: C1, C11, C12, C13, C2, C3, C4, C5, C6, C7, C8, J1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
