File: Electronique/Clavier/_autosave-pcb.kicad_sch (KiCad schematic)
At the start: 170 parts, among them J3 Conn_01x05, Q3 BSS84, Q4 BSS138, SW1 A, SW10 R, SW11 F, SW12 C, SW13 T, SW14 G, SW15 V, SW16 Y, SW17 H, SW18 B, SW19 1, SW2 Q, SW20 2, SW21 3, SW22 4, SW23 5, SW24 6, SW25 7, SW26 U, SW27 J, SW28 N, SW29 8, SW3 <, SW30 I, SW31 K, SW32 ,, SW33 9, SW34 O, SW35 L, SW36 ;, SW37 0, SW38 P, SW39 M, SW4 Z, SW40 :, SW41 SW_Push, SW42 SW_Push, SW43 ², SW44 Tab, SW45 VMaj, SW46 Shift, SW47 Echap, SW48 F1, SW49 F2, SW5 S, SW50 F3, SW51 F4, SW52 F5, SW53 F6, SW54 F7, SW55 F8, SW56 F9, SW57 F10, SW58 F11, SW59 ), SW6 W, SW60 ^, SW61 ù, SW62 !, SW63 F12, SW64 =, SW65 $, SW66 *, SW67 Up, SW7 E, SW8 D, SW9 X, U1 ESP32-S3-WROOM-1, U3 USBLC6-2P6, U4 TLV75533PDBV, U6 MCP73871-2CC

Commit message: update keyboard schematic
Parts:
- added C10, C9: 10nF, Capacitor_SMD:C_0603_1608Metric_Pad1.08x0.95mm_HandSolder, symbol Device:C
- added R1: 10K, symbol Device:R
- added SW68: SW_Push_SPDT, symbol Switch:SW_Push_SPDT
- J3: footprint Connector_PinHeader_2.54mm:PinHeader_1x05_P2.54mm_Vertical -> Connector_PinHeader_2.54mm:PinHeader_1x05_P2.54mm_Horizontal
Connections:
- net +3.3V: now also R1.1
- net CLK: now also C9.1
- net DT: now also C10.1
- net GND: now also J2.S1 (SHIELD), C10.2, C9.2
- net Vbat: now also SW68.1 (A); no longer J1.2 (Pin_2)
- net PG: now reaches D71.1 (K), U6.6 (~{PG})
- net PG: now also U1.9 (IO16), R1.2
- new net: J1.2 (Pin_2), SW68.2 (B)
- no-connect marks 3 -> 2
Other:
- note added: "Mesure de la batterie"
- note removed: "Circuit de vérification de la capacité de la batterie L'ADC de l'ESP32 étant limité à une tension de 3,3V, un PDT par 0,68 est utilisé pour ramener la tension batterie (max 4,2V) à 2,88v max. Le transistor NMOS est controlé par le µC pour décider quand on veut vérifier la capacité de la batterie. Le transistor PMOS coupe l'alimentation du PDT et est controlé par le NMOS, donc le µC, évitant ainsi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"
- note removed: "Indicateur de batterie"
- note removed: "Note : Le régulateur TLV75533PDBV à un dropout Maximum de 238mV, il faut donc qu'il soit alimenté au minimum en 3v5 pour fournir du 3v3."
- moved on the sheet: J1
