File: Electronique/Clavier/µC_ESP32/_autosave-clavier.kicad_sch (KiCad schematic)
At the start: 46 parts, among them J4 Conn_02x13_Odd_Even, Q1 2N7002, Q2 SI2365EDS, SW74 SW_Push_SPDT, U1 USBLC6-2P6, U2 MCP73871-2CC, U4 ESP32-S3-WROOM-1

Commit message: global update
Connections:
- net Col10: now also U4.33 (IO40); no longer U4.25 (IO48)
