File: Electronique/Clavier/µC_ESP32/clavier.kicad_sch (KiCad schematic)
At the start: 46 parts, among them J4 Conn_02x13_Odd_Even, Q1 2N7002, Q2 SI2365EDS, SW74 SW_Push_SPDT, U1 USBLC6-2P6, U2 MCP73871-2CC, U4 ESP32-S3-WROOM-1

Commit message: mm
Parts:
- removed H1, H2, H3, H4: MountingHole_Pad, MountingHole:MountingHole_3.2mm_M3_DIN965_Pad, symbol Mechanical:MountingHole_Pad
- removed J1: ~, Connector_USB:USB_C_Receptacle_G-Switch_GT-USB-7010ASV, symbol Connector:USB_C_Receptacle_USB2.0_16P
- removed J4: Conn_02x13_Odd_Even, Connector_IDC:IDC-Header_2x13_P2.54mm_Vertical, symbol Connector_Generic:Conn_02x13_Odd_Even
- added J2: Conn_02x13_Odd_Even, Connector_PinHeader_2.54mm:PinHeader_2x13_P2.54mm_Vertical, symbol Connector_Generic:Conn_02x13_Odd_Even
- added J4: USB_C_Receptacle_USB2.0_14P, Connector_USB:USB_C_Receptacle_XKB_U262-16XN-4BVC11, symbol Connector:USB_C_Receptacle_USB2.0_14P
- J3: renamed from J2; value ~ -> (none); footprint Connector_JST:JST_PH_B2B-PH-K_1x02_P2.00mm_Vertical -> Connector_JST:JST_PH_S2B-PH-K_1x02_P2.00mm_Horizontal
- R12: renamed from R16; value 100k -> 27k
- R13: renamed from R17; value 220k -> 68k
- Rprog1: renamed from R12; value 2k -> 3k3
- Rprog3: renamed from R11; value 20k -> 3k3
- U1: footprint Package_TO_SOT_SMD:SOT-666 -> Package_TO_SOT_SMD:SOT-23-6
- renumbered C9 to C10, C12 to C5, C13 to C6, C14 to C7, C15 to C8, C8 to C9, R21 to R10, R15 to R11, R4 to R3, R5 to R4, R6 to R5, R7 to R6, R9 to R7, R19 to R8, R20 to R9, R13 to Rtherm1, SW74 to SW1, U4 to U2, U2 to U3
Connections:
- net +3.3V: now also J2.22 (Pin_22)
- net Col1: now also J2.21 (Pin_21)
- net Col10: now also U2.33 (IO40), J2.3 (Pin_3); no longer U2.25 (IO48)
- net Col11: now also J2.2 (Pin_2)
- net Col12: now also J2.4 (Pin_4)
- net Col13: now also J2.6 (Pin_6)
- net Col14: now also J2.8 (Pin_8)
- net Col15: now also J2.10 (Pin_10)
- net Col2: now also J2.19 (Pin_19)
- net Col3: now also J2.17 (Pin_17)
- net Col4: now also J2.15 (Pin_15)
- net Col5: now also J2.13 (Pin_13)
- net Col6: now also J2.11 (Pin_11)
- net Col7: now also J2.9 (Pin_9)
- net Col8: now also J2.7 (Pin_7)
- net Col9: now also J2.5 (Pin_5)
- net D+: now also J4.A6 (D+), J4.B6 (D+)
- net D-: now also J4.A7 (D-), J4.B7 (D-)
- net GND: now also J3.2 (Pin_2), J2.14 (Pin_14), J2.18 (Pin_18), J4.A1 (GND), J4.A12 (GND), J4.B1 (GND), J4.B12 (GND), J4.SH (SHIELD); no longer J3.1 (Pin_1)
- net L1: now also J2.16 (Pin_16)
- net L2: now also J2.25 (Pin_25)
- net L3: now also J2.23 (Pin_23)
- net L4: now also J2.1 (Pin_1)
- net L5: now also J2.12 (Pin_12)
- net Mute_btn: now also J2.20 (Pin_20)
- net Vbat_Mes: now also J3.1 (Pin_1); no longer J3.2 (Pin_2)
- net Vol_Down: now also J2.26 (Pin_26)
- net Vol_Up: now also J2.24 (Pin_24)
- net at R1.1: now also J4.A5 (CC1)
- net at R2.1: now also J4.B5 (CC2)
- net Valim renamed VCC
- net Vbat+ renamed +BATT
- net Vusb renamed VBUS
- net VBUS: now also J4.A4 (VBUS), J4.A9 (VBUS), J4.B4 (VBUS), J4.B9 (VBUS); no longer U3.17 (CE)
- new net CE: U2.25 (IO48), U3.17 (CE)
- no-connect marks 8 -> 9
Other:
- moved on the sheet: C10, C4, C9, J3, R3, R4, R5, R6, R7, Rprog1, Rprog3, Rtherm1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
