File: Electronique/Clavier/Matrice/matrice.kicad_pcb (KiCad board)
At the start: 2 copper layers, 300.5 x 95.5 mm, 150 parts, among them J1 Conn_02x13_Odd_Even, SW10 Win, SW11 2, SW12 Z, SW13 S, SW14 W, SW15 Alt, SW16 3, SW17 E, SW18 D, SW19 X, SW2 Tab, SW20 4, SW21 R, SW22 F, SW23 C, SW24 5, SW25 T, SW26 G, SW27 V, SW28 Space, SW29 6, SW3 VMaj, SW30 Y, SW31 H, SW32 B, SW33 7, SW34 U, SW35 J, SW36 N, SW37 COM-15141, SW38 8, SW39 I, SW4 Shift, SW40 K, SW41 ,, SW42 9, SW43 O, SW44 L, SW45 ;, SW46 0, SW47 P, SW48 M, SW49 :, SW5 CTRL, SW50 R5, SW51 ), SW52 ^, SW53 ù, SW54 !, SW55 R6, SW56 =, SW57 $, SW58 *, SW59 PageUp, SW6 1, SW60 Left, SW61 Delete, SW62 Up, SW63 Down, SW64 Entrer, SW65 Definir, SW66 Supp, SW67 PageDown, SW68 Right, SW7 A, SW70 Fn, SW71 S1, SW72 S2, SW73 R4, SW8 Q, SW9 <

Commit message: mm
Parts:
- J1: moved to B.Cu
- moved J1 2.62 mm to (72.8, 123.0), turned to 0 degrees
Connections:
- J1 pad 1: L4 -> Col11
- J1 pad 10: Col15 -> Col7
- J1 pad 11: Col6 -> L5
- J1 pad 12: L5 -> Col6
- J1 pad 13: Col5 -> GND
- J1 pad 14: GND -> Col5
- J1 pad 15: Col4 -> L1
- J1 pad 16: L1 -> Col4
- J1 pad 17: Col3 -> GND
- J1 pad 18: GND -> Col3
- J1 pad 19: Col2 -> Mute_btn
- J1 pad 2: Col11 -> L4
- J1 pad 20: Mute_btn -> Col2
- J1 pad 21: Col1 -> +3.3V
- J1 pad 22: +3.3V -> Col1
- J1 pad 23: L3 -> Vol_Up
- J1 pad 24: Vol_Up -> L3
- J1 pad 25: L2 -> Vol_Down
- J1 pad 26: Vol_Down -> L2
- J1 pad 3: Col10 -> Col12
- J1 pad 4: Col12 -> Col10
- J1 pad 5: Col9 -> Col13
- J1 pad 6: Col13 -> Col9
- J1 pad 7: Col8 -> Col14
- J1 pad 8: Col14 -> Col8
- J1 pad 9: Col7 -> Col15
- SW37 pad 1: GND -> unconnected-(SW37-Pad1)
- SW37 pad 2: GND -> unconnected-(SW37-Pad2)
- SW37 pad 4: GND -> unconnected-(SW37-Pad4)
