File: Electronique/Clavier/Matrice/matrice.kicad_sch (KiCad schematic)
At the start: 150 parts, among them J1 Conn_02x13_Odd_Even, SW10 Win, SW11 2, SW12 Z, SW13 S, SW14 W, SW15 Alt, SW16 3, SW17 E, SW18 D, SW19 X, SW2 Tab, SW20 4, SW21 R, SW22 F, SW23 C, SW24 5, SW25 T, SW26 G, SW27 V, SW28 Space, SW29 6, SW3 VMaj, SW30 Y, SW31 H, SW32 B, SW33 7, SW34 U, SW35 J, SW36 N, SW37 COM-15141, SW38 8, SW39 I, SW4 Shift, SW40 K, SW41 ,, SW42 9, SW43 O, SW44 L, SW45 ;, SW46 0, SW47 P, SW48 M, SW49 :, SW5 CTRL, SW50 R5, SW51 ), SW52 ^, SW53 ù, SW54 !, SW55 R6, SW56 =, SW57 $, SW58 *, SW59 PageUp, SW6 1, SW60 Left, SW61 Delete, SW62 Up, SW63 Down, SW64 Entrer, SW65 Definir, SW66 Supp, SW67 PageDown, SW68 Right, SW7 A, SW70 Fn, SW71 S1, SW72 S2, SW73 R4, SW8 Q, SW9 <

Commit message: mm
Connections:
- net +3.3V: now also J1.21 (Pin_21); no longer J1.22 (Pin_22)
- net Col1: now also J1.22 (Pin_22); no longer J1.21 (Pin_21)
- net Col10: now also J1.4 (Pin_4); no longer J1.3 (Pin_3)
- net Col11: now also J1.1 (Pin_1); no longer J1.2 (Pin_2)
- net Col12: now also J1.3 (Pin_3); no longer J1.4 (Pin_4)
- net Col13: now also J1.5 (Pin_5); no longer J1.6 (Pin_6)
- net Col14: now also J1.7 (Pin_7); no longer J1.8 (Pin_8)
- net Col15: now also J1.9 (Pin_9); no longer J1.10 (Pin_10)
- net Col2: now also J1.20 (Pin_20); no longer J1.19 (Pin_19)
- net Col3: now also J1.18 (Pin_18); no longer J1.17 (Pin_17)
- net Col4: now also J1.16 (Pin_16); no longer J1.15 (Pin_15)
- net Col5: now also J1.14 (Pin_14); no longer J1.13 (Pin_13)
- net Col6: now also J1.12 (Pin_12); no longer J1.11 (Pin_11)
- net Col7: now also J1.10 (Pin_10); no longer J1.9 (Pin_9)
- net Col8: now also J1.8 (Pin_8); no longer J1.7 (Pin_7)
- net Col9: now also J1.6 (Pin_6); no longer J1.5 (Pin_5)
- net GND: now also J1.13 (Pin_13), J1.17 (Pin_17); no longer J1.14 (Pin_14), J1.18 (Pin_18), SW37.1, SW37.2, SW37.4
- net L1: now also J1.15 (Pin_15); no longer J1.16 (Pin_16)
- net L2: now also J1.26 (Pin_26); no longer J1.25 (Pin_25)
- net L3: now also J1.24 (Pin_24); no longer J1.23 (Pin_23)
- net L4: now also J1.2 (Pin_2); no longer J1.1 (Pin_1)
- net L5: now also J1.11 (Pin_11); no longer J1.12 (Pin_12)
- net Mute_btn: now also J1.19 (Pin_19); no longer J1.20 (Pin_20)
- net Vol_Down: now also J1.25 (Pin_25); no longer J1.26 (Pin_26)
- net Vol_Up: now also J1.23 (Pin_23); no longer J1.24 (Pin_24)
- no-connect marks 0 -> 3
Other:
- moved on the sheet: J1, R3
