File: Electronique/Dongle/dongle.kicad_pcb (KiCad board)
At the start: 2 copper layers, 27.6 x 18.3 mm, 15 parts, among them J1 USB_A, SW3 SW_Push, SW4 SW_Push, U1 USBLC6-2P6, U2 ESP32-S3-MINI-1-N8, U4 TLV75533PDBV

Commit message: update
Parts:
- removed C1, C2, C5: 10µ, Capacitor_SMD:C_0603_1608Metric_Pad1.08x0.95mm_HandSolder
- removed U4: TLV75533PDBV, Package_TO_SOT_SMD:SOT-23-5
- added C3: 10µ, Capacitor_SMD:C_0603_1608Metric_Pad1.08x0.95mm_HandSolder, F.Cu at (213.3, 100.7)
- added C4: 10µ, Capacitor_SMD:C_0603_1608Metric_Pad1.08x0.95mm_HandSolder, F.Cu at (213.1, 94.1)
- added C8: 100n, Capacitor_SMD:C_0603_1608Metric_Pad1.08x0.95mm_HandSolder, F.Cu at (212.9, 92.5)
- added PS1: BU33SD5WG-TR, MyFootprints:SOT95P280X125-5N, F.Cu at (214.3, 97.0)
- SW3: value SW_Push -> BOOT; footprint Button_Switch_SMD:SW_Tactile_SPST_NO_Straight_CK_PTS636Sx25SMTRLFS -> MyFootprints:434771025826
- SW4: value SW_Push -> RST; footprint Button_Switch_SMD:SW_Tactile_SPST_NO_Straight_CK_PTS636Sx25SMTRLFS -> MyFootprints:434771025826
- U2: footprint ESP32-S3-MINI:ESP32-S3-MINI-1-N8 -> MyFootprints:ESP32-S3-MINI-1-N8
- moved D4 2.05 mm to (223.5, 98.4), turned to 90 degrees
- moved C7 1.82 mm to (221.9, 95.8)
- moved SW3 1.64 mm to (216.6, 104.7)
- moved R3 1.59 mm to (221.5, 98.6), turned to 90 degrees
- moved R5 1.58 mm to (218.2, 97.2)
- moved SW4 0.46 mm to (218.7, 92.7)
Connections:
- net 5V renamed +5V
Routing:
- net +5V: track 18.3 -> 23.5 mm
- net +3.3V: track 22.3 -> 23.1 mm
- net GND: vias 1 -> 6
Other:
- board text added: "Axel"
- board text added: "Bottom"
- board text added: "Top"

Commit message: mm
Parts:
- moved J1 8.59 mm to (191.4, 98.5)
- moved C4 5.61 mm to (207.7, 92.8), turned to 180 degrees
- moved C8 5.57 mm to (207.7, 94.3), turned to 180 degrees
- moved SW3 1.89 mm to (214.9, 103.8)
- moved C3 1.35 mm to (211.9, 100.7)
- moved PS1 1.35 mm to (213.0, 97.0)
- moved U1 0.81 mm to (206.9, 98.4)
Routing:
- net +3.3V: track 23.1 -> 0.04 mm, vias 3 -> 0
- net +5V: track 23.5 -> 6.37 mm
- net EN (Reset): track 13.7 -> 2.19 mm
- net BOOT: track 6.91 -> 0.00 mm
- net D-: track 3.12 -> 0.00 mm
- net D+: track 3.10 -> 0.00 mm, vias 1 -> 0
- net Net-(D4-A): track 1.99 -> 0.01 mm
- net DP-: track 1.81 -> 2.82 mm
- net DP+: track 1.82 -> 2.82 mm
- net GND: vias 6 -> 5
Other:
- board size 27.6 x 18.3 mm -> 34.9 x 18.3 mm
- board text removed: "Bottom"
