File: Electronique/Dongle/dongle.kicad_sch (KiCad schematic)
At the start: 15 parts, among them J1 USB_A, SW3 SW_Push, SW4 SW_Push, U1 USBLC6-2P6, U2 ESP32-S3-MINI-1-N8, U4 TLV75533PDBV

Commit message: update
Parts:
- removed C1, C2, C5: 10µ, Capacitor_SMD:C_0603_1608Metric_Pad1.08x0.95mm_HandSolder, symbol Device:C
- removed U4: TLV75533PDBV, Package_TO_SOT_SMD:SOT-23-5, symbol Regulator_Linear:TLV75533PDBV
- added C3, C4: 10µ, Capacitor_SMD:C_0603_1608Metric_Pad1.08x0.95mm_HandSolder, symbol Device:C
- added C8: 100n, Capacitor_SMD:C_0603_1608Metric_Pad1.08x0.95mm_HandSolder, symbol Device:C
- added PS1: BU33SD5WG-TR, MyFootprints:SOT95P280X125-5N, symbol BU33SD5WG-TR:BU33SD5WG-TR
- SW3: value SW_Push -> BOOT; footprint Button_Switch_SMD:SW_Tactile_SPST_NO_Straight_CK_PTS636Sx25SMTRLFS -> MyFootprints:434771025826
- SW4: value SW_Push -> RST; footprint Button_Switch_SMD:SW_Tactile_SPST_NO_Straight_CK_PTS636Sx25SMTRLFS -> MyFootprints:434771025826
- U2: footprint ESP32-S3-MINI:ESP32-S3-MINI-1-N8 -> MyFootprints:ESP32-S3-MINI-1-N8
Connections:
- net +3.3V: now also C4.1, C8.1, PS1.5 (VOUT)
- net GND: now also C3.2, C4.2, C8.2, PS1.2 (GND)
- net 5V renamed +5V
- net +5V: now also C3.1, PS1.1 (VIN), PS1.3 (STBY)
- no-connect marks 0 -> 34
Other:
- moved on the sheet: D4, R3, R4, R5, U1

Commit message: mm
Parts:
- U1: footprint Package_TO_SOT_SMD:SOT-666 -> Package_TO_SOT_SMD:SOT-23-6
